File: mp3.sch (KiCad schematic (older format))
At the start: 9 parts

Commit message: Updated schematic
Parts:
- removed U?: ADP2503, symbol mp3:ADP2503
- added C?: 2.2u, symbol Device:C
- added C?: 20u, symbol Device:C
- added C?: 10u, symbol Device:C
- added L?: 2uH, symbol Device:L
- added R?: 24K, symbol Device:R
- added R?: 3k, symbol Device:R
- added R?: 320k, symbol Device:R
- added R?: 40k, symbol Device:R
- added U?: ADP2503, symbol mp3:ADP2503
- C?: value 4.7uF -> 4.7u
- C?: value 2.2uF -> 10u
Connections:
- wire segments 23 -> 56
Other:
- moved on the sheet: C?, D?, J?, R?, U?

Commit message: Updated values on resistor divider for ADP2503 to adjust output to 4.0V assuming 4.2 in
Parts:
- R?: value 320k -> 330K
- R?: value 40k -> 47K
Changed lines of the file:
@@
 P 5200 2650
 F 0 "R?" H 5270 2696 50  0000 L CNN
-F 1 "320k" H 5270 2605 50  0000 L CNN
+F 1 "330K" H 5270 2605 50  0000 L CNN
 F 2 "" V 5130 2650 50  0001 C CNN
 F 3 "~" H 5200 2650 50  0001 C CNN
@@
 P 5200 3050
 F 0 "R?" H 5270 3096 50  0000 L CNN
-F 1 "40k" H 5270 3005 50  0000 L CNN
+F 1 "47K" H 5270 3005 50  0000 L CNN
 F 2 "" V 5130 3050 50  0001 C CNN
 F 3 "~" H 5200 3050 50  0001 C CNN
